Commit message: working version

File: my_robot_description/urdf/camera.xacro (robot description, xacro)
@@ -15,5 +15,5 @@
         <child link="camera_optical_frame"/>
         <!-- Mounted 6cm forward on top deck -->
-        <origin xyz="0.125 0 ${camera_elevation}" rpy="-1.570796327 0 -1.570796327"/>
+        <origin xyz="0.013 0 ${camera_elevation}" rpy="-1.570796327 0 -1.570796327"/>
     </joint>
     <!-- Link: Frame ID used by ROS 2 /scan message -->

File: my_robot_description/urdf/chassis.xacro (robot description, xacro)
@@ -17,5 +17,5 @@
     <!-- =================================================================== -->
     <xacro:property name="chassis_length" value="0.250"/> <!-- 25 cm -->
-    <xacro:property name="chassis_width"  value="0.180"/> <!-- 18 cm -->
+    <xacro:property name="chassis_width"  value="0.20"/> <!-- 18 cm -->
     <xacro:property name="chassis_height" value="0.1075"/> <!-- 6 cm 0.060-->
     <xacro:property name="chassis_mass"   value="0.800"/> <!-- 800 g -->
@@ -23,9 +23,9 @@
     <xacro:property name="wheel_thickness" value="0.026"/> <!-- 26 mm width -->
     <xacro:property name="wheel_mass"      value="0.050"/> <!-- 50 g -->
-    <xacro:property name="wheel_offset_y"  value="0.105"/> <!-- Track width center-to-wheel -->
-    <xacro:property name="wheel_offset_x"  value="0.11"/> <!-- Axle position along length -->
+    <xacro:property name="wheel_offset_y"  value="0.1165"/> <!-- Track width center-to-wheel -->
+    <xacro:property name="wheel_offset_x"  value="0.0"/> <!-- Axle position along length -->
     <xacro:property name="caster_radius"  value="0.015"/> <!-- 30 mm caster ball -->
     <xacro:property name="caster_mass"    value="0.030"/>
-    <xacro:property name="caster_offset_x" value="-0.080"/> <!-- Front/rear caster position -->
+    <xacro:property name="caster_offset_x" value="-0.185"/> <!-- Front/rear caster position -->
     <!-- =================================================================== -->
     <!-- 1. BASE FOOTPRINT (Ground plane z=0) -->
@@ -42,5 +42,5 @@
     <link name="base_link">
         <visual>
-            <origin xyz="0 0 ${chassis_height/2}" rpy="0 0 0"/>
+            <origin xyz="-0.105 0 ${chassis_height/2}" rpy="0 0 0"/>
             <geometry>
                 <box size="${chassis_length} ${chassis_width} ${chassis_height}"/>
@@ -49,5 +49,5 @@
         </visual>
         <collision>
-            <origin xyz="0 0 ${chassis_height/2}" rpy="0 0 0"/>
+            <origin xyz="-0.105 0 ${chassis_height/2}" rpy="0 0 0"/>
             <geometry>
                 <box size="${chassis_length} ${chassis_width} ${chassis_height}"/>
@@ -55,5 +55,5 @@
         </collision>
         <xacro:inertial_box mass="${chassis_mass}" x="${chassis_length}" y="${chassis_width}" z="${chassis_height}">
-            <origin xyz="0 0 ${chassis_height/2}" rpy="0 0 0"/>
+            <origin xyz="-0.105 0 ${chassis_height/2}" rpy="0 0 0"/>
         </xacro:inertial_box>
     </link>

File: my_robot_description/urdf/mobile_microbot.xacro (robot description, xacro)
@@ -5,5 +5,5 @@
     <joint name="arm_base_joint" type="fixed"> <parent link="base_link" />
         <child link="link0" />
-        <origin xyz="0.072 0.0 0.0965" rpy="0 0 -1.5708" />
+        <origin xyz="-0.037 0.0 0.0965" rpy="0 0 -1.5708" />
     </joint>
 </robot>
