Commit message: adding nanobot files

File: my_robot_description/urdf/arm.urdf (robot description, URDF)
Before this commit: robot microbot, 12 links, 11 joints
Links:
- added link tcp_link
Joints:
- added joint wrist_to_tcp: type fixed, parent wrist, child tcp_link, origin xyz=0.0 0.0 0.08 rpy=0 0 0
- joint joint1: limit lower=-3.14158 upper=3.14158 effort=100 velocity=100 -> lower=-1.570796327 upper=1.570796327 effort=100 velocity=100
- joint joint2: limit lower=-3.14158 upper=3.14158 effort=100 velocity=100 -> lower=-2.617993878 upper=0.523598776 effort=100 velocity=100
- joint joint3: limit lower=-3.14158 upper=3.14158 effort=100 velocity=100 -> lower=-2.617993878 upper=0.523598776 effort=100 velocity=100
- joint joint4: limit lower=-3.14158 upper=3.14158 effort=100 velocity=100 -> lower=-2.617993878 upper=0.523598776 effort=100 velocity=100
- joint wrist_joint: limit lower=-3.14158 upper=3.14158 effort=100 velocity=100 -> lower=-1.570796327 upper=1.570796327 effort=100 velocity=100

Commit message: NonoBot modifications

File: my_robot_description/urdf/arm.urdf (robot description, URDF)
Before this commit: robot microbot, 13 links, 12 joints
Links:
- link link0: geometry collision mesh filename=package://my_robot_description/meshes/link0.stl scale=0.001 0.001 0.001; visual mesh filename=package://my_robot_description/meshes/link0.stl scale=0.001 0.001 0.001
- link link1: geometry collision mesh filename=package://my_robot_description/meshes/link1.stl scale=0.001 0.001 0.001; visual mesh filename=package://my_robot_description/meshes/link1.stl scale=0.001 0.001 0.001
- link link2: geometry collision mesh filename=package://my_robot_description/meshes/link2.stl scale=0.001 0.001 0.001; visual mesh filename=package://my_robot_description/meshes/link2.stl scale=0.001 0.001 0.001
- link link3: geometry collision mesh filename=package://my_robot_description/meshes/link3.stl scale=0.001 0.001 0.001; visual mesh filename=package://my_robot_description/meshes/link3.stl scale=0.001 0.001 0.001
- link link4: mass 0.798614 -> None; geometry 
- link wrist: mass 0.05 -> None; geometry 
Joints:
- joint joint1: origin xyz=0 0 0.012 rpy=0 0 0 -> xyz=0 0 0.0 rpy=0 0 0
- joint joint2: origin xyz=0 -0.040505 0.126375 rpy=0 0 0 -> xyz=0 0.0405055 0.133875 rpy=0 0 0
- joint joint3: origin xyz=0 0.0 0.116 rpy=0.0 0 0 -> xyz=0 0.0 0.165188 rpy=0.0 0 0
- joint joint4: axis 1 0 0 -> (none); limit lower=-2.617993878 upper=0.523598776 effort=100 velocity=100 -> (none); origin xyz=0 0.0 0.135 rpy=0.0 0 0 -> xyz=0 0.0 0.117188 rpy=0.0 0 0; type revolute -> fixed
- joint robot_joint7: origin xyz=0 0 0.0065 rpy=0 0 0 -> xyz=0 0 0.0 rpy=0 0 0
- joint wrist_joint: axis 0 0 1 -> (none); limit lower=-1.570796327 upper=1.570796327 effort=100 velocity=100 -> (none); origin xyz=0.0 0.0 0.104 rpy=0 0 0 -> xyz=0.0 0.0 0.0 rpy=0 0 0; type revolute -> fixed

File: my_robot_description/urdf/mobile_nanobot.xacro (robot description, xacro)
@@ -1,9 +1,9 @@
 <?xml version="1.0"?>
-<robot name="mobile_microbot" xmlns:xacro="http://ros.org/wiki/xacro">
+<robot name="mobile_nanobot" xmlns:xacro="http://ros.org/wiki/xacro">
     <xacro:include filename="$(find my_robot_description)/urdf/robot.urdf.xacro" />
     <xacro:include filename="$(find my_robot_description)/urdf/arm.urdf" />
     <joint name="arm_base_joint" type="fixed"> <parent link="base_link" />
         <child link="link0" />
-        <origin xyz="-0.037 0.0 0.0965" rpy="0 0 -1.5708" />
+        <origin xyz="0.032 0.0 0.1085" rpy="0 0 -1.5708" />
     </joint>
 </robot>

File: nanobot_moveit_config/config/mobile_nanobot.ros2_control.xacro (robot description, xacro)
@@ -1,5 +1,5 @@
 <?xml version="1.0"?>
 <robot xmlns:xacro="http://www.ros.org/wiki/xacro">
-    <xacro:macro name="mobile_microbot_ros2_control" params="name initial_positions_file">
+    <xacro:macro name="mobile_nanobot_ros2_control" params="name initial_positions_file">
         <xacro:property name="initial_positions" value="${load_yaml(initial_positions_file)['initial_positions']}"/>
         <ros2_control name="${name}" type="system">
